File: _hw/zynqAIO_Baro.sch (KiCad schematic (older format))
At the start: 4 parts

Commit message: Removed Zybo board part. Not needed and complicates project setup.
Configured DDR3 to 16-bit width (using only 1 of the 2 DDR3 chips on Zybo but aligned more to zynqFC configuration).

Disabled Ethernet/USB. Not part of zynqFC.

Enabled SPI0 peripheral for IMU, I²C1 peripheral for EEPROM and UART0 peripheral for GPS.
However, all three interfaces cannot be used on Zybo and will not be used in SW.

Updated HW pinning to current Zynq PS bank planning.
Changed lines of the file:
@@
 	4200 3900 4200 3800
 Wire Wire Line
-	4050 3800 4900 3800
+	4050 3800 4200 3800
 Wire Wire Line
 	4350 3800 4350 3750
@@
 Connection ~ 4050 3400
 Wire Wire Line
-	4900 3400 3900 3400
+	4900 3400 4800 3400
 Wire Wire Line
 	4900 3700 4800 3700
@@
 	5900 3000 5900 2900
 Wire Wire Line
-	5600 3400 6300 3400
+	5600 3400 5900 3400
 Wire Wire Line
 	5900 3400 5900 3300
@@
 Text Notes 7300 3750 0    60   ~ 0
 to Zynq\nPL bank\n35
+Wire Wire Line
+	4800 3400 4350 3400
+Wire Wire Line
+	4350 3800 4800 3800
+Wire Wire Line
+	4200 3800 4350 3800
+Wire Wire Line
+	4350 3400 4050 3400
+Wire Wire Line
+	4050 3400 3900 3400
+Wire Wire Line
+	4800 3800 4900 3800
+Wire Wire Line
+	5900 3400 6300 3400
 $EndSCHEMATC
