File: _hw/zynqAIO_GPS.sch (KiCad schematic (older format))
At the start: 9 parts

Commit message: Removed Zybo board part. Not needed and complicates project setup.
Configured DDR3 to 16-bit width (using only 1 of the 2 DDR3 chips on Zybo but aligned more to zynqFC configuration).

Disabled Ethernet/USB. Not part of zynqFC.

Enabled SPI0 peripheral for IMU, I²C1 peripheral for EEPROM and UART0 peripheral for GPS.
However, all three interfaces cannot be used on Zybo and will not be used in SW.

Updated HW pinning to current Zynq PS bank planning.
Changed lines of the file:
@@
 	6550 3650 6550 3600
 Wire Wire Line
-	6550 3300 6550 3200
+	6550 3300 6550 3250
 Wire Wire Line
 	6550 2900 6550 2850
@@
 	6550 3250 6200 3250
 Wire Wire Line
-	6200 3250 6200 3800
+	6200 3250 6200 3650
 Connection ~ 6550 3250
 Wire Wire Line
@@
 $EndComp
 Wire Wire Line
-	4850 3650 5050 3650
+	4850 3650 4950 3650
 Wire Wire Line
 	4950 3650 4950 3500
@@
 $EndComp
 Wire Wire Line
-	4450 3500 4450 3800
+	4450 3500 4450 3650
 Wire Wire Line
 	4450 3800 5050 3800
@@
 Wire Wire Line
 	5050 4100 4350 4100
+Wire Wire Line
+	6550 3250 6550 3200
+Wire Wire Line
+	6200 3650 6200 3800
+Wire Wire Line
+	4950 3650 5050 3650
+Wire Wire Line
+	4450 3650 4450 3800
 $EndSCHEMATC
