File: _hw/zynqAIO_IMU.sch (KiCad schematic (older format))
At the start: 8 parts, among them U701 BMX160

Commit message: Removed Zybo board part. Not needed and complicates project setup.
Configured DDR3 to 16-bit width (using only 1 of the 2 DDR3 chips on Zybo but aligned more to zynqFC configuration).

Disabled Ethernet/USB. Not part of zynqFC.

Enabled SPI0 peripheral for IMU, I²C1 peripheral for EEPROM and UART0 peripheral for GPS.
However, all three interfaces cannot be used on Zybo and will not be used in SW.

Updated HW pinning to current Zynq PS bank planning.
Connections:
- net IMU_INT3: now reaches U?.12 (INT)
Changed lines of the file:
@@
 	3300 3200 3850 3200
 Wire Wire Line
-	3300 3300 3850 3300
+	3300 3300 3600 3300
 Wire Wire Line
 	3300 3400 3850 3400
@@
 	3000 4150 3000 4100
 Wire Wire Line
-	2800 4100 3850 4100
+	2800 4100 3000 4100
 Connection ~ 3000 4100
 Wire Wire Line
@@
 	3750 4200 3750 4550
 Wire Wire Line
-	2800 4550 3850 4550
+	2800 4550 3000 4550
 Connection ~ 3750 4550
 Wire Wire Line
@@
 $EndComp
 Wire Wire Line
-	7300 3750 7800 3750
+	7300 3750 7500 3750
 Wire Wire Line
 	7500 3750 7500 3300
@@
 $EndComp
 Wire Wire Line
-	8500 2550 8500 3050
-Wire Wire Line
-	8500 2650 9400 2650
+	8500 2550 8500 2650
+Wire Wire Line
+	8500 2650 9000 2650
 Wire Wire Line
 	9400 2650 9400 2700
@@
 	9200 3100 9200 3050
 Wire Wire Line
-	9000 3050 9400 3050
+	9000 3050 9200 3050
 Wire Wire Line
 	9000 3050 9000 3000
@@
 Text Notes 6100 3750 0    60   ~ 0
 to Zynq\nPS bank\n501
+Wire Wire Line
+	3600 3300 3850 3300
+Wire Wire Line
+	3000 4100 3350 4100
+Wire Wire Line
+	3350 4100 3800 4100
+Wire Wire Line
+	3800 4100 3850 4100
+Wire Wire Line
+	3750 4550 3850 4550
+Wire Wire Line
+	3350 4550 3750 4550
+Wire Wire Line
+	3000 4550 3350 4550
+Wire Wire Line
+	7500 3750 7800 3750
+Wire Wire Line
+	9000 2650 9400 2650
+Wire Wire Line
+	8500 2650 8500 3050
+Wire Wire Line
+	9200 3050 9400 3050
+Text GLabel 9500 3450 2    60   Input ~ 0
+IMU_INT3
+Wire Wire Line
+	9200 3450 9500 3450
 $EndSCHEMATC
