File: _hw/zynqAIO_RAM.sch (KiCad schematic (older format))
At the start: 24 parts, among them U801 DDR3-SDRAM-96FBGA

Commit message: Removed Zybo board part. Not needed and complicates project setup.
Configured DDR3 to 16-bit width (using only 1 of the 2 DDR3 chips on Zybo but aligned more to zynqFC configuration).

Disabled Ethernet/USB. Not part of zynqFC.

Enabled SPI0 peripheral for IMU, I²C1 peripheral for EEPROM and UART0 peripheral for GPS.
However, all three interfaces cannot be used on Zybo and will not be used in SW.

Updated HW pinning to current Zynq PS bank planning.
Other:
- note added: "Micron MT41J128M16JT-125"
Changed lines of the file:
@@
 Wire Wire Line
 	6650 5100 7050 5100
+Text Notes 2650 1500 0    50   ~ 0
+ Micron MT41J128M16JT-125
 $EndSCHEMATC
