File: _hw/zynqAIO_ROM.sch (KiCad schematic (older format))
At the start: 12 parts, among them J601 Micro_SD_Card, U601 S25FL128S, U602 24AA02

Commit message: Removed Zybo board part. Not needed and complicates project setup.
Configured DDR3 to 16-bit width (using only 1 of the 2 DDR3 chips on Zybo but aligned more to zynqFC configuration).

Disabled Ethernet/USB. Not part of zynqFC.

Enabled SPI0 peripheral for IMU, I²C1 peripheral for EEPROM and UART0 peripheral for GPS.
However, all three interfaces cannot be used on Zybo and will not be used in SW.

Updated HW pinning to current Zynq PS bank planning.
Changed lines of the file:
@@
 	2450 2150 2950 2150
 Wire Wire Line
-	2450 2300 2950 2300
+	2450 2300 2600 2300
 Wire Wire Line
 	2450 2450 2950 2450
@@
 	2850 1450 2850 1350
 Wire Wire Line
-	2000 3300 2950 3300
+	2000 3300 2250 3300
 Wire Wire Line
 	2950 3450 2900 3450
@@
 	2950 3600 2900 3600
 Wire Wire Line
-	2900 3600 2900 3800
-Wire Wire Line
-	2250 3700 2900 3700
+	2900 3600 2900 3700
+Wire Wire Line
+	2250 3700 2600 3700
 Wire Wire Line
 	2600 3700 2600 3650
@@
 	6750 2650 6750 3500
 Wire Wire Line
-	6750 3500 5900 3500
+	6750 3500 6550 3500
 Wire Wire Line
 	6350 3950 6350 3900
 Wire Wire Line
-	6150 3900 6900 3900
+	6150 3900 6350 3900
 Wire Wire Line
 	6150 3900 6150 3850
@@
 $EndComp
 Wire Wire Line
-	2250 5700 3100 5700
-Wire Wire Line
-	2250 5900 3100 5900
+	2250 5700 2600 5700
+Wire Wire Line
+	2250 5900 2800 5900
 Wire Wire Line
 	2600 5700 2600 5600
@@
 	2600 5300 2600 5200
 Wire Wire Line
-	2600 5200 4350 5200
+	2600 5200 2800 5200
 Wire Wire Line
 	2800 5300 2800 5200
@@
 Text Notes 1050 5950 0    60   ~ 0
 to Zynq\nPS bank \n501
+Wire Wire Line
+	2600 2300 2950 2300
+Wire Wire Line
+	2900 3300 2950 3300
+Wire Wire Line
+	2900 3700 2900 3800
+Wire Wire Line
+	2600 3300 2900 3300
+Wire Wire Line
+	2600 3700 2900 3700
+Wire Wire Line
+	2250 3300 2600 3300
+Wire Wire Line
+	6350 3900 6550 3900
+Wire Wire Line
+	6150 3500 5900 3500
+Wire Wire Line
+	6550 3500 6150 3500
+Wire Wire Line
+	6550 3900 6900 3900
+Wire Wire Line
+	2600 5700 3100 5700
+Wire Wire Line
+	2800 5900 3100 5900
+Wire Wire Line
+	2800 5200 3050 5200
+Wire Wire Line
+	3050 5200 3500 5200
+Wire Wire Line
+	3500 5200 4350 5200
 $EndSCHEMATC

Commit message: Added text note about EEPROM chip device
Other:
- note added: "Microchip 24AA02E48"
Changed lines of the file:
@@
 Wire Wire Line
 	3500 5200 4350 5200
+Text Notes 3150 5100 0    50   ~ 0
+Microchip 24AA02E48
 $EndSCHEMATC
